Commit message: DH with URDF

File: urdf/turret.urdf (robot description, URDF)
Before this commit: robot turret, 6 links, 5 joints
Joints:
- joint joint2: axis 0 0 -1 -> 0 0 1; origin xyz=0. 0 0.0 rpy=-1.57 0 0 -> xyz=0. 0 0.0 rpy=1.57079632679 0 0
- joint joint3: origin xyz=0. -0.05 0. rpy=1.57 0 0 -> xyz=0. 0 0. rpy=-1.57079632679 0 0
- joint link4_2: origin xyz=0.0 0 0.05 rpy=0 0 0 -> xyz=0.0 0 0.1 rpy=0 0 0
