Commit message: debug dh_code.py

File: urdf/scara.urdf (robot description, URDF)
Before this commit: robot scara, 10 links, 9 joints
Joints:
- joint joint1: limit lower=-1.57 upper=1.57 effort=10 velocity=3 -> lower=-1.5707963267948 upper=1.5707963267948 effort=10 velocity=3
- joint joint2: limit lower=-1.57 upper=1.57 effort=10 velocity=3 -> lower=-1.5707963267948 upper=1.5707963267948 effort=10 velocity=3; origin xyz=0.2 0 0.045 rpy=0 0 1.57 -> xyz=0.2 0 0.045 rpy=0 0 1.5707963267948
- joint joint3: limit lower=-1.57 upper=1.57 effort=10 velocity=3 -> lower=-1.5707963267948 upper=1.5707963267948 effort=10 velocity=3; origin xyz=0. -.15 0.0 rpy=1.57 0 0 -> xyz=0. -.15 0.0 rpy=1.5707963267948 0 0
- joint joint4: origin xyz=0. -0.07 0.0 rpy=1.57 0 0 -> xyz=0. -0.07 0.0 rpy=1.5707963267948 0 0

Commit message: fix to dh_code for Ubuntu 18.04

File: urdf/scara.urdf (robot description, URDF)
Before this commit: robot scara, 10 links, 9 joints
Links:
- link end_effector: mass 1.0 -> None
- link link2_2: mass 1.0 -> None
- link link4: mass 1.0 -> None
